File: Kicad/ESP01-Programmer.kicad_pcb (KiCad board)
At the start: 2 copper layers, 80 x 20.3 mm, 6 parts, among them J1 Power Connector, J2 FTDI, U1 ESP-01v090

Commit message: V1.1: Adding I2C bus headers.
More information and resources are also added.
Parts:
- added J3: I2C, Connector_PinHeader_2.54mm:PinHeader_1x02_P2.54mm_Vertical, F.Cu at (85.1, 38.1)
- added J4: I2C, Connector_PinHeader_2.54mm:PinHeader_1x02_P2.54mm_Vertical, F.Cu at (85.1, 41.9)
- added R3: 10K, Resistor_THT:R_Axial_DIN0207_L6.3mm_D2.5mm_P10.16mm_Horizontal, F.Cu at (91.4, 35.6)
Connections:
- net Net-(JP1-Pad2) renamed SDA
- net Net-(R1-Pad2) renamed SCL
Routing:
- net SCL: track 23.7 -> 65.6 mm
- net SDA: track 49.8 -> 65.4 mm
- net VCC: track 95.3 -> 96.6 mm
Other:
- board text added: "SCL"
- board text added: "SDA"
